File: hardware/mega-seedy.kicad_pcb (KiCad board)
At the start: 2 copper layers, 19 parts, among them J1 Conn_01x03_Male, M1 Motor_DC, M2 Motor_DC, M3 Motor_DC, U1 ChinaBluePill, U2 L9110, U3 L9110, U4 4N25, U5 4N25, U6 4N25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

Commit message: schematic updated for sensor arrays, comms, etc
Parts:
- M1: value Motor_DC -> Steer Motor
- M2: value Motor_DC -> Drive Motors
- M3: value Motor_DC -> Back Mtr
Other:
- board text added: "3V3"
- board text added: "9V"
- board text added: "GND"
Changed lines of the file:
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@@
   (general
     (thickness 1.6)
-    (drawings 0)
+    (drawings 4)
     (tracks 111)
     (zones 0)
@@
   (page A4)
   (layers
-    (0 F.Cu signal)
+    (0 F.Cu signal hide)
     (31 B.Cu signal)
     (32 B.Adhes user)
@@
       (effects (font (size 1 1) (thickness 0.15)))
     )
-    (fp_text value Motor_DC (at 2.54 1.27 180) (layer F.Fab)
+    (fp_text value "Steer Motor" (at 2.54 1.27 180) (layer F.SilkS)
       (effects (font (size 1 1) (thickness 0.15)))
     )
@@
       (effects (font (size 1 1) (thickness 0.15)))
     )
-    (fp_text value Motor_DC (at 0 4.87 180) (layer F.Fab)
+    (fp_text value "Drive Motors" (at -2.54 5.08 180) (layer F.SilkS)
       (effects (font (size 1 1) (thickness 0.15)))
     )
@@
       (effects (font (size 1 1) (thickness 0.15)))
     )
-    (fp_text value Motor_DC (at 0 4.87 180) (layer F.Fab)
+    (fp_text value "Back Mtr" (at 0 4.87 180) (layer F.Fab) hide
       (effects (font (size 1 1) (thickness 0.15)))
     )
@@
     )
   )
+  (gr_text 3V3 (at 96.52 36.83) (layer F.SilkS)
+    (effects (font (size 1 1) (thickness 0.25)))
+  )
+  (gr_text GND (at 101.6 36.83) (layer F.SilkS)
+    (effects (font (size 1 1) (thickness 0.25)))
+  )
+  (gr_text GND (at 99.06 35.56) (layer F.Cu)
+    (effects (font (size 1.5 1.5) (thickness 0.3)))
+  )
+  (gr_text 9V (at 91.44 36.83) (layer F.SilkS)
+    (effects (font (size 1 1) (thickness 0.25)))
+  )
   (segment (start 81.28 33.02) (end 82.55 31.75) (width 0.5) (layer F.Cu) (net 1))
