File: hardware/mega-seedy.sch (KiCad schematic (older format))
At the start: 19 parts, among them J1 Conn_01x03_Male, M1 Motor_DC, M2 Motor_DC, M3 Motor_DC, U1 ChinaBluePill, U2 L9110, U3 L9110, U4 4N25, U5 4N25, U6 4N25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

Commit message: schematic updated for sensor arrays, comms, etc
Parts:
- added D1, D2, D3, D4, D5: D, Diode_THT:D_DO-15_P2.54mm_Vertical_AnodeUp, symbol Device:D
- added M4, M5: Motor_Servo, Connector_PinHeader_2.54mm:PinHeader_1x03_P2.54mm_Vertical, symbol Motor:Motor_Servo
- added U10, U11, U12, U13, U9: HC-SR04, Connector_PinHeader_2.54mm:PinHeader_1x04_P2.54mm_Vertical, symbol HC-SR04:HC-SR04
- added U14: VL53L1X_Breakout, Connector_PinHeader_2.54mm:PinHeader_2x03_P2.54mm_Vertical, symbol misc:VL53L1X_Breakout
- added U15: NEO6M_Breakout, symbol misc:NEO6M_Breakout
- added U8: NRF24L01_Breakout, RF_Module:nRF24L01_Breakout, symbol RF:NRF24L01_Breakout
- added U?: L3GD20+LSM303D_Breakout, symbol misc:L3GD20+LSM303D_Breakout
Connections:
- net +3V3: now also M4.2 (+), M5.2 (+), U10.1 (VCC), U11.1 (VCC), U12.1 (VCC), U13.1 (VCC), U14.1 (VIN), U15.1 (VCC), U8.2 (VCC), U8.3 (CE), U9.1 (VCC), U?.2 (3Vo)
- net GND: now also M4.3 (-), M5.3 (-), U10.4 (GND), U11.4 (GND), U12.4 (GND), U13.4 (GND), U14.2 (GND), U15.2 (GND), U8.1 (GND), U8.4 (~CSN), U9.4 (GND), U?.3 (GND)
- net REV: now reaches U7.1
- net REV: now also U1.PA0; no longer U1.PA11
- net FWD: now reaches U6.1
- net FWD: now also U1.PA1; no longer U1.PA10
- net RIGHT: now reaches U5.1
- net RIGHT: now also U1.PA2; no longer U1.PA9
- net LEFT: now reaches U4.1
- net LEFT: now also U1.PA3; no longer U1.PA8
- net at M2.1 (+), M3.1 (+): now also U3.4 (OB); no longer U3.1 (OA)
- net at M2.2 (-), M3.2 (-): now also U3.1 (OA); no longer U3.4 (OB)
- net TRIG1: now reaches U1.PA12
- net TRIG1: now also U9.2 (TRIG)
- net ECHO: now reaches U1.PA15
- net ECHO: now also D1.1 (K), D2.1 (K), D3.1 (K), D4.1 (K), D5.1 (K)
- net IRQ: now reaches U1.PA4
- net IRQ: now also U8.8 (IRQ)
- net SCK: now reaches U1.PA5
- net SCK: now also U8.5 (SCK)
- net MISO: now reaches U1.PA6
- net MISO: now also U8.7 (MISO)
- net MOSI: now reaches U1.PA7
- net MOSI: now also U8.6 (MOSI)
- net GRXD: now reaches U1.PB10
- net GRXD: now also U15.3 (RXD)
- net GTXD: now reaches U1.PB11
- net GTXD: now also U15.4 (TXD)
- net GPPS: now reaches U1.PB12
- net GPPS: now also U15.5 (PPS)
- net PITCH: now reaches U1.PB4
- net PITCH: now also M4.1 (PWM)
- net YAW: now reaches U1.PB5
- net YAW: now also M5.1 (PWM)
- net GPIO1: now reaches U1.PB6
- net GPIO1: now also U14.5 (GPIO1)
- net XSHUT: now reaches U1.PB7
- net XSHUT: now also U14.6 (XSHUT)
- net SDA: now reaches U1.PB8
- net SDA: now also U14.4 (SDA), U?.5 (SDA)
- net SCL: now reaches U1.PB9
- net SCL: now also U14.3 (SCL), U?.4 (SCL)
- new net: D1.2 (A), U9.3 (ECHO)
- new net: D2.2 (A), U10.3 (ECHO)
- new net: D3.2 (A), U11.3 (ECHO)
- new net: D4.2 (A), U12.3 (ECHO)
- new net: D5.2 (A), U13.3 (ECHO)
- new net TRIG2: U1.PA11, U10.2 (TRIG)
- new net TRIG3: U1.PA10, U11.2 (TRIG)
- new net TRIG4: U1.PA9, U12.2 (TRIG)
- new net TRIG5: U1.PA8, U13.2 (TRIG)
- no-connect marks 35 -> 22
Other:
- note added: "Drive Control"
- note added: "Fixed Proximity Sensor Array"
- note added: "Gimbal Mount LIDAR"
- note added: "Navigation"
- note added: "Power Connection"
- note added: "Steering Control"
- moved on the sheet: J1, M1, M2, M3, R1, R2, R3, R4, R5, R6, R7, R8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
